File: kicad/Particulate_matters/_autosave-Particulate_matters.kicad_sch (KiCad schematic)
At the start: 4 parts, among them U1 XIAO-ESP32-S3-DIP

Commit message: Updated schematic and pcb design
Parts:
- added U5: ~, symbol ParticulateMatters:SSD1306_128x32_0.91
Connections:
- net GND: now also U5.1 (GND)
- net VCC: now also U5.2 (VCC)
- net at U1.5 (GPIO5/D4/I2C_SDA), U3.3 (SDA): now also U5. (SDA)
- net at U1.6 (GPIO9/D5/I2C_SCL), U3.4 (SDL): now also U5.3 (SCK)
Changed lines of the file:
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@@
 	(generator_version "9.0")
 	(paper "A4")
+	(junction
+		(at 104.14 99.06)
+		(diameter 0)
+		(color 0 0 0 0)
+	)
+	(junction
+		(at 101.6 95.25)
+		(diameter 0)
+		(color 0 0 0 0)
+	)
 	(wire
 		(pts
@@
 	(wire
 		(pts
+			(xy 161.29 111.76) (xy 101.6 111.76)
+		)
+		(stroke
+			(width 0)
+			(type default)
+		)
+	)
+	(wire
+		(pts
 			(xy 161.29 76.2) (xy 194.31 76.2)
 		)
@@
 	(wire
 		(pts
+			(xy 153.67 100.33) (xy 161.29 100.33)
+		)
+		(stroke
+			(width 0)
+			(type default)
+		)
+	)
+	(wire
+		(pts
+			(xy 153.67 104.14) (xy 161.29 104.14)
+		)
+		(stroke
+			(width 0)
+			(type default)
+		)
+	)
+	(wire
+		(pts
 			(xy 161.29 68.58) (xy 175.26 68.58)
 		)
@@
 	(wire
 		(pts
+			(xy 101.6 111.76) (xy 101.6 95.25)
+		)
+		(stroke
+			(width 0)
+			(type default)
+		)
+	)
+	(wire
+		(pts
 			(xy 170.18 83.82) (xy 170.18 80.01)
 		)
@@
 	(wire
 		(pts
+			(xy 161.29 107.95) (xy 104.14 107.95)
+		)
+		(stroke
+			(width 0)
+			(type default)
+		)
+	)
+	(wire
+		(pts
 			(xy 161.29 72.39) (xy 194.31 72.39)
 		)
@@
 	(wire
 		(pts
+			(xy 104.14 107.95) (xy 104.14 99.06)
+		)
+		(stroke
+			(width 0)
+			(type default)
+		)
+	)
+	(wire
+		(pts
 			(xy 175.26 68.58) (xy 175.26 80.01)
 		)
@@
 	(hierarchical_label "GND"
 		(shape input)
+		(at 153.67 100.33 180)
+		(effects
+			(font
+				(size 1.27 1.27)
+			)
+			(justify right)
+		)
+	)
+	(hierarchical_label "GND"
+		(shape input)
 		(at 74.93 60.96 0)
 		(effects
@@
 			)
 			(justify left)
+		)
+	)
+	(hierarchical_label "VCC"
+		(shape input)
+		(at 153.67 104.14 180)
+		(effects
+			(font
+				(size 1.27 1.27)
+			)
+			(justify right)
 		)
 	)
@@
 					(unit 1)
 				)
+			)
+		)
+	)
+	(symbol
+		(lib_id "ParticulateMatters:SSD1306_128x32_0.91")
+		(at 226.06 96.52 0)
+		(mirror y)
+		(unit 1)
+		(exclude_from_sim no)
+		(in_bom yes)
+		(on_board yes)
+		(dnp no)
+		(fields_autoplaced yes)
+		(property "Reference" "U5"
+			(at 227.33 104.7721 0)
+			(effects
+				(font
+					(size 1.27 1.27)
+				)
+				(justify right)
+			)
+		)
+		(property "Value" "~"
+			(at 227.33 106.6772 0)
+			(effects
+				(font
+					(size 1.27 1.27)
+				)
+				(justify right)
+			)
+		)
+		(property "Footprint" ""
+			(at 226.06 96.52 0)
+			(effects
+				(font
+					(size 1.27 1.27)
+				)
+				(hide yes)
+			)
+		)
+		(property "Datasheet" ""
+			(at 226.06 96.52 0)
+			(effects
+				(font
+					(size 1.27 1.27)
+				)
+				(hide yes)
+			)
+		)
+		(property "Description" ""
+			(at 226.06 96.52 0)
+			(effects
+				(font
+					(size 1.27 1.27)
+				)
+				(hide yes)
+			)
+		)
+		(pin "2"
+		)
+		(pin "1"
+		)
+		(pin "3"
+		)
+		(pin ""
+		)
+		(instances
+			(project ""
+				(path "/a469de4a-6558-4c6c-9733-dd68d37b40f4"
+					(reference "U5")
+					(unit 1)
+				)
